File: PCB/hackypad.kicad_sch (KiCad schematic)
At the start: 0 parts

Commit message: feat(PCB): Create PCB schematic
Parts:
- added D1, D2, D3, D4, D5, D6, D7, D8, D9: 1N4148, Diode_THT:D_DO-35_SOD27_P7.62mm_Horizontal, symbol Diode:1N4148
- added J1: Conn_01x04, symbol Connector_Generic:Conn_01x04
- added SW1, SW2, SW3, SW4, SW5, SW6, SW7, SW8, SW9: SW_Push_45deg, symbol Switch:SW_Push_45deg
- added SW10: RotaryEncoder_Switch, symbol Device:RotaryEncoder_Switch
- added U1: MOUDLE-SEEEDUINO-XIAO, symbol XIAO_RP2040:MOUDLE-SEEEDUINO-XIAO
- added U2: ER_OLEDM0.91_1x-I2C, Display:ER_OLEDM0.91_1x-I2C, symbol Display_Graphic:ER_OLEDM0.91_1x-I2C
Connections:
- new net: D4.2 (A), SW4.2
- new net: D2.2 (A), SW2.2
- new net: D8.2 (A), SW8.2
- new net: D6.2 (A), SW6.2
- new net: D1.2 (A), SW1.2
- new net: D3.2 (A), SW3.2
- new net: D7.2 (A), SW7.2
- new net: D9.2 (A), SW9.2
- new net: D5.2 (A), SW5.2
- new net Col 0: SW1.1, SW4.1, SW7.1, U1.4 (PA11_A3_D3)
- new net Col 1: SW2.1, SW5.1, SW8.1, U1.7 (PB08_A6_D6_TX)
- new net Col 2: SW3.1, SW6.1, SW9.1, U1.8 (PB09_A7_D7_RX)
- new net Encoder A: SW10.A, U1.11 (PA6_A10_D10_MOSI)
- new net Encoder B: SW10.B, U1.10 (PA5_A9_D9_MISO)
- new net Encoder Sw: SW10.S1, U1.9 (PA7_A8_D8_SCK)
- new net GND: SW10.C, SW10.S2, U1.13 (GND), U2.1 (GND)
- new net Row 0: D1.1 (K), D2.1 (K), D3.1 (K), U1.1 (PA02_A0_D0)
- new net Row 1: D4.1 (K), D5.1 (K), D6.1 (K), U1.2 (PA4_A1_D1)
- new net Row 2: D7.1 (K), D8.1 (K), D9.1 (K), U1.3 (PA10_A2_D2)
- new net SCL: U1.6 (PA9_A5_D5_SCL), U2.3 (SCL)
- new net SDA: U1.5 (PA8_A4_D4_SDA), U2.4 (SDA)
- new net VCC: U1.12 (3V3), U2.2 (VCC)

Commit message: feat(PCB): Add footprints
Parts:
- removed J1: Conn_01x04, symbol Connector_Generic:Conn_01x04
- SW1, SW2, SW3, SW4, SW5, SW6, SW7, SW8, SW9: footprint (none) -> Button_Switch_Keyboard:SW_Cherry_MX_1.00u_PCB
- SW10: footprint (none) -> Rotary_Encoder:RotaryEncoder_Alps_EC11E-Switch_Vertical_H20mm
- U1: footprint (none) -> footprints:XIAO-Generic-Hybrid-14P-2.54-21X17.8MM
Connections:
- no-connect marks 0 -> 1
Changed lines of the file:
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@@
 		(color 0 0 0 0)
 	)
+	(no_connect
+		(at 74.93 78.74)
+	)
 	(wire
 		(pts
@@
 			)
 		)
-		(property "Footprint" ""
+		(property "Footprint" "Button_Switch_Keyboard:SW_Cherry_MX_1.00u_PCB"
 			(at 137.16 106.68 0)
 			(hide yes)
@@
 			)
 		)
-		(property "Footprint" ""
+		(property "Footprint" "Button_Switch_Keyboard:SW_Cherry_MX_1.00u_PCB"
 			(at 153.67 83.82 0)
 			(hide yes)
@@
 			)
 		)
-		(property "Footprint" ""
+		(property "Footprint" "Button_Switch_Keyboard:SW_Cherry_MX_1.00u_PCB"
 			(at 170.18 106.68 0)
 			(hide yes)
@@
 			)
 		)
-		(property "Footprint" ""
+		(property "Footprint" "Button_Switch_Keyboard:SW_Cherry_MX_1.00u_PCB"
 			(at 137.16 83.82 0)
 			(hide yes)
@@
 			)
 		)
-		(property "Footprint" ""
+		(property "Footprint" "Button_Switch_Keyboard:SW_Cherry_MX_1.00u_PCB"
 			(at 170.18 129.54 0)
 			(hide yes)
@@
 			)
 		)
-		(property "Footprint" ""
+		(property "Footprint" "footprints:XIAO-Generic-Hybrid-14P-2.54-21X17.8MM"
 			(at 36.83 83.82 0)
 			(hide yes)
@@
 			)
 		)
-		(property "Footprint" ""
+		(property "Footprint" "Button_Switch_Keyboard:SW_Cherry_MX_1.00u_PCB"
 			(at 170.18 83.82 0)
 			(hide yes)
@@
 	)
 	(symbol
-		(lib_id "Connector_Generic:Conn_01x04")
-		(at 43.18 40.64 0)
-		(unit 1)
-		(body_style 1)
-		(exclude_from_sim no)
-		(in_bom yes)
-		(on_board yes)
-		(in_pos_files yes)
-		(dnp no)
-		(fields_autoplaced yes)
-		(property "Reference" "J1"
-			(at 45.72 40.6399 0)
-			(show_name no)
-			(do_not_autoplace no)
-			(effects
-				(font
-					(size 1.27 1.27)
-				)
-				(justify left)
-			)
-		)
-		(property "Value" "Conn_01x04"
-			(at 45.72 43.1799 0)
-			(show_name no)
-			(do_not_autoplace no)
-			(effects
-				(font
-					(size 1.27 1.27)
-				)
-				(justify left)
-			)
-		)
-		(property "Footprint" ""
-			(at 43.18 40.64 0)
-			(hide yes)
-			(show_name no)
-			(do_not_autoplace no)
-			(effects
-				(font
-					(size 1.27 1.27)
-				)
-			)
-		)
-		(property "Datasheet" ""
-			(at 43.18 40.64 0)
-			(hide yes)
-			(show_name no)
-			(do_not_autoplace no)
-			(effects
-				(font
-					(size 1.27 1.27)
-				)
-			)
-		)
-		(property "Description" "Generic connector, single row, 01x04, script generated (kicad-library-utils/schlib/autogen/connector/)"
-			(at 43.18 40.64 0)
-			(hide yes)
-			(show_name no)
-			(do_not_autoplace no)
-			(effects
-				(font
-					(size 1.27 1.27)
-				)
-			)
-		)
-		(pin "4"
-		)
-		(pin "1"
-		)
-		(pin "2"
-		)
-		(pin "3"
-		)
-		(instances
-			(project "hackypad"
-				(path "/cd7e2b5b-f4a5-4b1a-b875-467cdf3ca38f"
-					(reference "J1")
-					(unit 1)
-				)
-			)
-		)
-	)
-	(symbol
 		(lib_id "Device:RotaryEncoder_Switch")
 		(at 99.06 53.34 0)
@@
 			)
 		)
-		(property "Footprint" ""
+		(property "Footprint" "Rotary_Encoder:RotaryEncoder_Alps_EC11E-Switch_Vertical_H20mm"
 			(at 95.25 49.276 0)
 			(hide yes)
@@
 			)
 		)
-		(property "Footprint" ""
+		(property "Footprint" "Button_Switch_Keyboard:SW_Cherry_MX_1.00u_PCB"
 			(at 153.67 129.54 0)
 			(hide yes)
@@
 			)
 		)
-		(property "Footprint" ""
+		(property "Footprint" "Button_Switch_Keyboard:SW_Cherry_MX_1.00u_PCB"
 			(at 153.67 106.68 0)
 			(hide yes)
@@
 			)
 		)
-		(property "Footprint" ""
+		(property "Footprint" "Button_Switch_Keyboard:SW_Cherry_MX_1.00u_PCB"
 			(at 137.16 129.54 0)
 			(hide yes)

Commit message: feat(PCB): Add 3d models
Parts:
- SW1, SW2, SW3, SW4, SW5, SW6, SW7, SW8, SW9: footprint Button_Switch_Keyboard:SW_Cherry_MX_1.00u_PCB -> switch:SW_Cherry_MX_1.00u_PCB
Other:
- moved on the sheet: U2
Changed lines of the file:
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@@
 	(global_label "SDA"
 		(shape input)
-		(at 50.8 29.21 180)
+		(at 41.91 41.91 180)
 		(fields_autoplaced yes)
 		(effects
@@
 		)
 		(property "Intersheetrefs" "${INTERSHEET_REFS}"
-			(at 44.2467 29.21 0)
+			(at 35.3567 41.91 0)
 			(hide yes)
 			(show_name no)
@@
 	(global_label "SCL"
 		(shape input)
-		(at 50.8 24.13 180)
+		(at 41.91 36.83 180)
 		(fields_autoplaced yes)
 		(effects
@@
 		)
 		(property "Intersheetrefs" "${INTERSHEET_REFS}"
-			(at 44.3072 24.13 0)
+			(at 35.4172 36.83 0)
 			(hide yes)
 			(show_name no)
@@
 	(symbol
 		(lib_id "power:VCC")
-		(at 60.96 16.51 0)
+		(at 52.07 29.21 0)
 		(unit 1)
 		(body_style 1)
@@
 		(fields_autoplaced yes)
 		(property "Reference" "#PWR05"
-			(at 60.96 20.32 0)
+			(at 52.07 33.02 0)
 			(hide yes)
 			(show_name no)
@@
 		)
 		(property "Value" "VCC"
-			(at 60.96 11.43 0)
+			(at 52.07 24.13 0)
 			(show_name no)
 			(do_not_autoplace no)
@@
 		)
 		(property "Footprint" ""
-			(at 60.96 16.51 0)
+			(at 52.07 29.21 0)
 			(hide yes)
 			(show_name no)
@@
 		)
 		(property "Datasheet" ""
-			(at 60.96 16.51 0)
+			(at 52.07 29.21 0)
 			(hide yes)
 			(show_name no)
@@
 		)
 		(property "Description" "Power symbol creates a global label with name \"VCC\""
-			(at 60.96 16.51 0)
+			(at 52.07 29.21 0)
 			(hide yes)
 			(show_name no)
@@
 			)
 		)
-		(property "Footprint" "Button_Switch_Keyboard:SW_Cherry_MX_1.00u_PCB"
+		(property "Footprint" "switch:SW_Cherry_MX_1.00u_PCB"
 			(at 137.16 106.68 0)
 			(hide yes)
@@
 	(symbol
 		(lib_id "power:GND")
-		(at 60.96 36.83 0)
+		(at 52.07 49.53 0)
 		(unit 1)
 		(body_style 1)
@@
 		(fields_autoplaced yes)
 		(property "Reference" "#PWR04"
-			(at 60.96 43.18 0)
+			(at 52.07 55.88 0)
 			(hide yes)
 			(show_name no)
@@
 		)
 		(property "Value" "GND"
-			(at 60.96 41.91 0)
+			(at 52.07 54.61 0)
 			(show_name no)
 			(do_not_autoplace no)
@@
 		)
 		(property "Footprint" ""
-			(at 60.96 36.83 0)
+			(at 52.07 49.53 0)
 			(hide yes)
 			(show_name no)
@@
 		)
 		(property "Datasheet" ""
-			(at 60.96 36.83 0)
+			(at 52.07 49.53 0)
 			(hide yes)
 			(show_name no)
@@
 		)
 		(property "Description" "Power symbol creates a global label with name \"GND\" , ground"
-			(at 60.96 36.83 0)
+			(at 52.07 49.53 0)
 			(hide yes)
 			(show_name no)
@@
 	(symbol
 		(lib_id "Display_Graphic:ER_OLEDM0.91_1x-I2C")
-		(at 60.96 26.67 0)
+		(at 52.07 39.37 0)
 		(unit 1)
 		(body_style 1)
@@
 		(fields_autoplaced yes)
 		(property "Reference" "U2"
-			(at 69.85 25.3999 0)
+			(at 60.96 38.0999 0)
 			(show_name no)
 			(do_not_autoplace no)
@@
 		)
 		(property "Value" "ER_OLEDM0.91_1x-I2C"
-			(at 69.85 27.9399 0)
+			(at 60.96 40.6399 0)
 			(show_name no)
 			(do_not_autoplace no)
@@
 		)
 		(property "Footprint" "Display:ER_OLEDM0.91_1x-I2C"
-			(at 78.994 39.37 0)
+			(at 70.104 52.07 0)
 			(hide yes)
 			(show_name no)
@@
 		)
 		(property "Datasheet" "https://www.buydisplay.com/download/manual/ER-OLEDM0.91-1_Datasheet.pdf"
-			(at 103.632 41.402 0)
+			(at 94.742 54.102 0)
 			(hide yes)
 			(show_name no)
@@
 		)
 		(property "Description" "SSD1306 OLED module, 0.91 inch, 128x32, I2C"
-			(at 87.63 43.434 0)
+			(at 78.74 56.134 0)
 			(hide yes)
 			(show_name no)
@@
 			)
 		)
-		(property "Footprint" "Button_Switch_Keyboard:SW_Cherry_MX_1.00u_PCB"
+		(property "Footprint" "switch:SW_Cherry_MX_1.00u_PCB"
 			(at 153.67 83.82 0)
 			(hide yes)
@@
 			)
 		)
-		(property "Footprint" "Button_Switch_Keyboard:SW_Cherry_MX_1.00u_PCB"
+		(property "Footprint" "switch:SW_Cherry_MX_1.00u_PCB"
 			(at 170.18 106.68 0)
 			(hide yes)
@@
 			)
 		)
-		(property "Footprint" "Button_Switch_Keyboard:SW_Cherry_MX_1.00u_PCB"
+		(property "Footprint" "switch:SW_Cherry_MX_1.00u_PCB"
 			(at 137.16 83.82 0)
 			(hide yes)
@@
 			)
 		)
-		(property "Footprint" "Button_Switch_Keyboard:SW_Cherry_MX_1.00u_PCB"
+		(property "Footprint" "switch:SW_Cherry_MX_1.00u_PCB"
 			(at 170.18 129.54 0)
 			(hide yes)
@@
 			)
 		)
-		(property "Footprint" "Button_Switch_Keyboard:SW_Cherry_MX_1.00u_PCB"
+		(property "Footprint" "switch:SW_Cherry_MX_1.00u_PCB"
 			(at 170.18 83.82 0)
 			(hide yes)
@@
 			)
 		)
-		(property "Footprint" "Button_Switch_Keyboard:SW_Cherry_MX_1.00u_PCB"
+		(property "Footprint" "switch:SW_Cherry_MX_1.00u_PCB"
 			(at 153.67 129.54 0)
 			(hide yes)
@@
 			)
 		)
-		(property "Footprint" "Button_Switch_Keyboard:SW_Cherry_MX_1.00u_PCB"
+		(property "Footprint" "switch:SW_Cherry_MX_1.00u_PCB"
 			(at 153.67 106.68 0)
 			(hide yes)
@@
 			)
 		)
-		(property "Footprint" "Button_Switch_Keyboard:SW_Cherry_MX_1.00u_PCB"
+		(property "Footprint" "switch:SW_Cherry_MX_1.00u_PCB"
 			(at 137.16 129.54 0)
 			(hide yes)

Commit message: feat(PCB): Rework the pcb
Parts:
- removed SW1: SW_Push_45deg, switch:SW_Cherry_MX_1.00u_PCB, symbol Switch:SW_Push_45deg
Connections:
- net Col 0: now also SW10.S1
- net GND: no longer SW10.S2
- net Encoder S2: now reaches D1.2 (A)
- net Encoder S2: now also SW10.S2
- net Encoder Sw: no longer names the net of U1.9 (PA7_A8_D8_SCK)
- net Encoder Sw: no longer SW10.S1
- no-connect marks 1 -> 2
Other:
- moved on the sheet: D1, D2, D3, D4, D5, D6, D7, D8, D9, SW2, SW3, SW4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
